File: hardware/pcb/whisli-sense.kicad_pcb (KiCad board)
At the start: 2 copper layers, 72 x 72 mm, 10 parts, among them J1 zasilanie 5-36 V, U1 ESP32-C3-Zero, U2 HMMD mmWave, U3 SHT3x, U4 SCD41, U5 BH1750 GY-302, U6 Pololu D36V6F5

Commit message: płytka: napis whis.li sense, wersja i oznaczenie zasilania na sitodruku
Other:
- board text added: "+"
- board text added: "5–36 V"
- board text added: "v1 2026-10"
- board text added: "whis.li sense"
- board text added: "−"
