File: hardware/pcb/whisli-sense.kicad_pcb (KiCad board)
At the start: 2 copper layers, 72 x 72 mm, 10 parts, among them J1 zasilanie 5-36 V, U1 ESP32-C3-Zero, U2 HMMD mmWave, U3 SHT3x, U4 SCD41, U5 BH1750 GY-302, U6 Pololu D36V6F5

Commit message: płytka: otwory odciążające przewód zasilania przy J1
Parts:
- added H4: , , F.Cu at (77.7, 105.0)
- added H5: , , F.Cu at (82.3, 105.0)
